File: three_little_words/three_little_words.kicad_pcb (KiCad board)
At the start: 2 copper layers, 91 parts, among them J1 Eurorack_Power, J10 Eurorack_Mono_Jack, J11 Eurorack_Mono_Jack, J12 Eurorack_Mono_Jack, J13 Eurorack_Mono_Jack, J14 Eurorack_Mono_Jack, J15 Conn_01x17_Female, J16 Conn_01x14_Female, J17 Conn_01x17_Male, J18 Conn_01x14_Male, J2 Eurorack_Mono_Jack, J3 Eurorack_Mono_Jack, J4 Eurorack_Mono_Jack, J5 Eurorack_Mono_Jack, J6 Eurorack_Mono_Jack, J7 Eurorack_Mono_Jack, J8 SSD1306_OLED_CONN, J9 Eurorack_Mono_Jack, Q1 2N3904, Q2 2N3904, Q3 2N3904, SW1 SW_Push, SW2 SW_Push, SW3 SW_Push, SW4 RotaryEncoder_Switch, SW5 RotaryEncoder_Switch, SW6 RotaryEncoder_Switch, U1 NE5532, U2 NE5532, U3 NE5532, U4 LM1117-3.3, U5 Pico, U6 L7805

Commit message: Adding circuitsss.
Parts:
- J15, J16: moved to B.Cu
- moved J14 251.5 mm to (271.1, 117.4), turned to 90 degrees
- moved SW5 242.1 mm to (254.9, 57.0), turned to -90 degrees
- moved SW6 240.0 mm to (273.6, 57.0), turned to -90 degrees
- moved J11 222.9 mm to (271.2, 107.1), turned to 90 degrees
- moved SW4 221.2 mm to (236.1, 57.0), turned to -90 degrees
- moved SW2 219.8 mm to (249.2, 17.6)
- moved J10 214.3 mm to (252.4, 107.1), turned to 90 degrees
- moved J3 213.5 mm to (252.4, 95.5), turned to 90 degrees
- moved J12 204.0 mm to (233.7, 117.4), turned to 90 degrees
- moved J7 203.1 mm to (271.1, 85.4), turned to 90 degrees
- moved SW3 199.4 mm to (259.2, 17.6)
- moved J13 198.3 mm to (252.4, 117.4), turned to 90 degrees
- moved J6 194.5 mm to (252.4, 85.4), turned to 90 degrees
- moved J4 194.4 mm to (271.1, 95.5), turned to 90 degrees
- moved J5 186.1 mm to (233.7, 85.4), turned to 90 degrees
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Other:
- board outline added: 128.7 x 108.5 mm

Commit message: Tried to sort circuit. Mixed success.
Parts:
- C13, C14, D1, D2, J1, U5, U6: moved to B.Cu
- J15: value Conn_01x17_Female -> Conn_01x14_Female; footprint Connector_PinSocket_2.54mm:PinSocket_1x17_P2.54mm_Vertical -> Connector_PinSocket_2.54mm:PinSocket_1x14_P2.54mm_Vertical
- J17: value Conn_01x17_Male -> Conn_01x14_Male; footprint Connector_PinHeader_2.54mm:PinHeader_1x17_P2.54mm_Vertical -> Connector_PinHeader_2.54mm:PinHeader_1x14_P2.54mm_Vertical
- U4: footprint Package_TO_SOT_SMD:SOT-223-3_TabPin2 -> Package_TO_SOT_THT:TO-220-3_Vertical; moved to B.Cu
- moved R21 241.0 mm to (255.0, 148.3)
- moved R19 234.3 mm to (255.4, 153.6)
- moved R20 213.4 mm to (223.5, 160.6), turned to 90 degrees
- moved Q3 207.1 mm to (261.4, 158.1)
- moved Q1 200.8 mm to (258.3, 157.4), turned to 180 degrees
- moved U2 190.4 mm to (151.5, 179.4), turned to 180 degrees
- moved J1 183.6 mm to (207.3, 111.3), turned to 90 degrees
- moved R4 178.9 mm to (164.3, 188.7), turned to 90 degrees
- moved R3 178.3 mm to (153.9, 178.3)
- moved R17 177.4 mm to (133.9, 181.1)
- moved Q2 174.5 mm to (222.5, 147.9)
- moved D1 173.8 mm to (200.7, 119.7), turned to 180 degrees
- moved R35 173.4 mm to (141.5, 177.8), turned to 180 degrees
- moved R34 169.3 mm to (153.9, 188.2)
- moved R14 167.0 mm to (161.5, 181.6), turned to 180 degrees
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Connections:
- J15 pad 13: FP_OLED_SCL -> FP_GND
- J15 pad 14: FP_OLED_SDA -> FP_3V3
- J16 pad 1: FP_ENC_CCW_1 -> FP_TOP_BTN_3
- J16 pad 10: FP_TOP_BTN_3 -> FP_ENC_CCW_2
- J16 pad 11: FP_TOP_BTN_2 -> FP_ENC_BTN_2
- J16 pad 12: FP_TOP_BTN_1 -> FP_ENC_CW_3
- J16 pad 13: FP_GND -> FP_ENC_CCW_3
- J16 pad 14: FP_3V3 -> FP_ENC_BTN_3
- J16 pad 2: FP_ENC_CW_1 -> FP_TOP_BTN_2
- J16 pad 3: FP_ENC_BTN_3 -> FP_TOP_BTN_1
- J16 pad 4: FP_ENC_CCW_2 -> FP_OLED_SDA
- J16 pad 5: FP_ENC_CW_2 -> FP_OLED_SCL
- J16 pad 6: FP_ENC_BTN_2 -> FP_ENC_CW_1
- J16 pad 7: FP_ENC_CCW_3 -> FP_ENC_CCW_1
- J16 pad 8: FP_ENC_CW_3 -> FP_ENC_BTN_1
- J16 pad 9: FP_ENC_BTN_1 -> FP_ENC_CW_2
- J17 pad 13: BP_OLED_SCL -> BP_GND
- J17 pad 14: BP_OLED_SDA -> BP_3V3
- J18 pad 1: BP_ENC_CCW_1 -> BP_ENC_CCW_3
- J18 pad 10: BP_ENC_CCW_3 -> BP_ENC_CCW_2
- J18 pad 11: BP_ENC_CCW_2 -> BP_ENC_BTN_2
- J18 pad 12: BP_ENC_CCW_1 -> BP_ENC_BTN_3
- J18 pad 13: BP_GND -> BP_ENC_CCW_3
- J18 pad 14: BP_3V3 -> BP_ENC_BTN_3
- J18 pad 2: BP_ENC_BTN_1 -> BP_ENC_CCW_2
- J18 pad 3: BP_ENC_BTN_3 -> BP_ENC_CCW_1
- J18 pad 4: BP_ENC_CCW_2 -> BP_OLED_SDA
- J18 pad 5: BP_ENC_BTN_2 -> BP_OLED_SCL
- J18 pad 6: BP_ENC_BTN_2 -> BP_ENC_BTN_1
- J18 pad 7: BP_ENC_CCW_3 -> BP_ENC_CCW_1
- J18 pad 8: BP_ENC_BTN_3 -> BP_ENC_BTN_1
- J18 pad 9: BP_ENC_BTN_1 -> BP_ENC_BTN_2
Other:
- board size 128.7 x 108.5 mm -> 127.6 x 108.5 mm

Commit message: Finishing 3lw schematic
Parts:
- added  : , winterbloom:MountingHole_M3_Slotted_Eurorack, F.Cu at (138.6, 17.5)
- added  : , winterbloom:MountingHole_M3_Slotted_Eurorack, F.Cu at (93.0, 140.0)
- added  : , winterbloom:MountingHole_M3_Slotted_Eurorack, F.Cu at (138.6, 140.0)
- added  : , winterbloom:MountingHole_M3_Slotted_Eurorack, F.Cu at (93.0, 17.5)
- moved R28 204.8 mm to (207.9, 67.6), turned to -90 degrees
- moved D6 203.4 mm to (211.2, 75.4), turned to 90 degrees
- moved R23 199.3 mm to (204.7, 67.6), turned to -90 degrees
- moved D5 196.6 mm to (208.6, 77.7), turned to 180 degrees
- moved D8 195.3 mm to (211.1, 54.7), turned to -90 degrees
- moved D7 191.6 mm to (200.8, 53.8), turned to 0 degrees
- moved D3 190.1 mm to (181.8, 72.5)
- moved D4 190.1 mm to (184.8, 80.2)
- moved R22 190.1 mm to (171.7, 79.7)
- moved R25 190.1 mm to (187.5, 79.8)
- moved R26 190.1 mm to (187.5, 72.9)
- moved R29 188.1 mm to (201.0, 56.4), turned to -90 degrees
- moved R27 186.3 mm to (201.5, 75.2), turned to 90 degrees
- moved R30 181.5 mm to (208.1, 64.0), turned to 90 degrees
- moved R24 179.7 mm to (204.7, 64.0), turned to 90 degrees
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Connections:
- C1 pad 1: GND -> BP_GND
- C13 pad 1: GND -> BP_GND
- C14 pad 2: GND -> BP_GND
- C2 pad 1: GND -> BP_GND
- C3 pad 1: GND -> BP_GND
- C4 pad 1: GND -> BP_GND
- C5 pad 1: GND -> BP_GND
- C6 pad 1: GND -> BP_GND
- D4 pad 2: GND -> BP_GND
- D6 pad 2: GND -> BP_GND
- D8 pad 2: GND -> BP_GND
- J1 pad 3: GND -> BP_GND
- J1 pad 4: GND -> BP_GND
- J1 pad 5: GND -> BP_GND
- J1 pad 6: GND -> BP_GND
- J1 pad 7: GND -> BP_GND
- J1 pad 8: GND -> BP_GND
- J2 pad S: Net-(J2-PadS) -> FP_GND
- J2 pad TN: Net-(J2-PadS) -> FP_GND
- J3 pad S: Net-(J3-PadS) -> FP_GND
- J3 pad TN: Net-(J3-PadS) -> FP_GND
- Q1 pad 1: GND -> BP_GND
- Q2 pad 1: GND -> BP_GND
- Q3 pad 1: GND -> BP_GND
- R26 pad 1: GND -> BP_GND
- R28 pad 1: GND -> BP_GND
- R30 pad 1: GND -> BP_GND
- U4 pad 1: GND -> BP_GND
- U5 pad 35: unconnected-(U5-Pad35) -> BP_3V3
- U6 pad 2: GND -> BP_GND
Routing:
- net FP_GND: track 0.00 -> 479.6 mm
- net BP_GND: track 0.00 -> 305.3 mm, vias 0 -> 2
- net BP_3V3: track 0.00 -> 151.2 mm
- net FP_3V3: track 0.00 -> 150.4 mm
- net -12V: track 0.00 -> 125.9 mm, vias 0 -> 6
- net Net-(C8-Pad2): track 0.00 -> 114.4 mm, vias 0 -> 8
- net BP_CV_IN_JACK_3: track 0.00 -> 109.8 mm
- net +12V: track 0.00 -> 94.9 mm, vias 0 -> 11
- net PICO_CV_OUT_3: track 0.00 -> 89.0 mm, vias 0 -> 2
- net PICO_CV_OFFSET_2: track 0.00 -> 87.0 mm, vias 0 -> 4
- net BP_ENC_CCW_1: track 0.00 -> 83.7 mm
- net PICO_CV_OUT_2: track 0.00 -> 81.5 mm, vias 0 -> 2
- net PICO_VOCT_OFFSET_2: track 0.00 -> 77.5 mm, vias 0 -> 1
- net PICO_CV_OFFSET_3: track 0.00 -> 76.7 mm, vias 0 -> 5
- net PICO_TRIG_IN_2: track 0.00 -> 73.0 mm
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Other:
- board size 127.6 x 108.5 mm -> 196.2 x 128.5 mm
