File: three_little_words/3lw_fp_and_bp_circuit.kicad_pcb (KiCad board)
At the start: 2 copper layers, 227.9 x 128.5 mm, 95 parts, among them J1 Eurorack_Power, J10 Eurorack_Mono_Jack, J11 Eurorack_Mono_Jack, J12 Eurorack_Mono_Jack, J13 Eurorack_Mono_Jack, J14 Eurorack_Mono_Jack, J15 Conn_01x14_Female, J16 Conn_01x14_Female, J17 Conn_01x14_Male, J18 Conn_01x14_Male, J2 Eurorack_Mono_Jack, J3 Eurorack_Mono_Jack, J4 Eurorack_Mono_Jack, J5 Eurorack_Mono_Jack, J6 Eurorack_Mono_Jack, J7 Eurorack_Mono_Jack, J8 SSD1306_OLED_CONN, J9 Eurorack_Mono_Jack, Q1 2N3904, Q2 2N3904, Q3 2N3904, SW1 SW_Push, SW2 SW_Push, SW3 SW_Push, SW4 RotaryEncoder_Switch, SW5 RotaryEncoder_Switch, SW6 RotaryEncoder_Switch, U1 NE5532, U2 NE5532, U3 NE5532, U4 LM1117-3.3, U5 Pico, U6 L7805

Commit message: Adding gerbers for first run of three little words.
Parts:
- removed  : , winterbloom:MountingHole_M3_Slotted_Eurorack (x4)
Routing:
- net BP_CV_OUT_1: track 4.02 -> 3.35 mm
Other:
- board size 227.9 x 128.5 mm -> 117.3 x 108.5 mm
